Commit message: improve fss_px4_sim launch and visualize

File: src/fss_px4_sim/model/iris.urdf (robot description, URDF)
Before this commit: robot iris, 7 links, 6 joints
Links:
- link base_link: geometry collision box size=0.47 0.47 0.11; visual mesh filename=package://fss_px4_sim/model/meshes/iris.stl scale=1 1 1
- link rotor_0: geometry collision cylinder length=0.005 radius=0.128; visual mesh filename=package://fss_px4_sim/model/meshes/iris_prop_ccw.stl scale=1 1 1
- link rotor_1: geometry collision cylinder length=0.005 radius=0.128; visual mesh filename=package://fss_px4_sim/model/meshes/iris_prop_ccw.stl scale=1 1 1
- link rotor_2: geometry collision cylinder length=0.005 radius=0.128; visual mesh filename=package://fss_px4_sim/model/meshes/iris_prop_cw.stl scale=1 1 1
- link rotor_3: geometry collision cylinder length=0.005 radius=0.128; visual mesh filename=package://fss_px4_sim/model/meshes/iris_prop_cw.stl scale=1 1 1

File: src/fss_px4_sim/model/iris_blue.urdf (robot description, URDF)
Before this commit: robot iris, 7 links, 6 joints
Links:
- link base_link: geometry collision box size=0.47 0.47 0.11; visual mesh filename=package://fss_px4_sim/model/meshes/iris.stl scale=1 1 1
- link rotor_0: geometry collision cylinder length=0.005 radius=0.128; visual mesh filename=package://fss_px4_sim/model/meshes/iris_prop_ccw.stl scale=1 1 1
- link rotor_1: geometry collision cylinder length=0.005 radius=0.128; visual mesh filename=package://fss_px4_sim/model/meshes/iris_prop_ccw.stl scale=1 1 1
- link rotor_2: geometry collision cylinder length=0.005 radius=0.128; visual mesh filename=package://fss_px4_sim/model/meshes/iris_prop_cw.stl scale=1 1 1
- link rotor_3: geometry collision cylinder length=0.005 radius=0.128; visual mesh filename=package://fss_px4_sim/model/meshes/iris_prop_cw.stl scale=1 1 1

File: src/fss_px4_sim/model/iris_green.urdf (robot description, URDF)
Before this commit: robot iris, 7 links, 6 joints
Links:
- link base_link: geometry collision box size=0.47 0.47 0.11; visual mesh filename=package://fss_px4_sim/model/meshes/iris.stl scale=1 1 1
- link rotor_0: geometry collision cylinder length=0.005 radius=0.128; visual mesh filename=package://fss_px4_sim/model/meshes/iris_prop_ccw.stl scale=1 1 1
- link rotor_1: geometry collision cylinder length=0.005 radius=0.128; visual mesh filename=package://fss_px4_sim/model/meshes/iris_prop_ccw.stl scale=1 1 1
- link rotor_2: geometry collision cylinder length=0.005 radius=0.128; visual mesh filename=package://fss_px4_sim/model/meshes/iris_prop_cw.stl scale=1 1 1
- link rotor_3: geometry collision cylinder length=0.005 radius=0.128; visual mesh filename=package://fss_px4_sim/model/meshes/iris_prop_cw.stl scale=1 1 1

File: src/fss_px4_sim/model/iris_grey.urdf (robot description, URDF)
Before this commit: robot iris, 7 links, 6 joints
Links:
- link base_link: geometry collision box size=0.47 0.47 0.11; visual mesh filename=package://fss_px4_sim/model/meshes/iris.stl scale=1 1 1
- link rotor_0: geometry collision cylinder length=0.005 radius=0.128; visual mesh filename=package://fss_px4_sim/model/meshes/iris_prop_ccw.stl scale=1 1 1
- link rotor_1: geometry collision cylinder length=0.005 radius=0.128; visual mesh filename=package://fss_px4_sim/model/meshes/iris_prop_ccw.stl scale=1 1 1
- link rotor_2: geometry collision cylinder length=0.005 radius=0.128; visual mesh filename=package://fss_px4_sim/model/meshes/iris_prop_cw.stl scale=1 1 1
- link rotor_3: geometry collision cylinder length=0.005 radius=0.128; visual mesh filename=package://fss_px4_sim/model/meshes/iris_prop_cw.stl scale=1 1 1

File: src/fss_px4_sim/model/iris_red.urdf (robot description, URDF)
Before this commit: robot iris, 7 links, 6 joints
Links:
- link base_link: geometry collision box size=0.47 0.47 0.11; visual mesh filename=package://fss_px4_sim/model/meshes/iris.stl scale=1 1 1
- link rotor_0: geometry collision cylinder length=0.005 radius=0.128; visual mesh filename=package://fss_px4_sim/model/meshes/iris_prop_ccw.stl scale=1 1 1
- link rotor_1: geometry collision cylinder length=0.005 radius=0.128; visual mesh filename=package://fss_px4_sim/model/meshes/iris_prop_ccw.stl scale=1 1 1
- link rotor_2: geometry collision cylinder length=0.005 radius=0.128; visual mesh filename=package://fss_px4_sim/model/meshes/iris_prop_cw.stl scale=1 1 1
- link rotor_3: geometry collision cylinder length=0.005 radius=0.128; visual mesh filename=package://fss_px4_sim/model/meshes/iris_prop_cw.stl scale=1 1 1
